File: Attenuator.kicad_sch (KiCad schematic)
At the start: 30 parts

Commit message: Routed PCB
Parts:
- removed D1: BAV199DW, Package_TO_SOT_SMD:SOT-363_SC-70-6, symbol Diode:BAV199DW
- added D2, D3: BAV199W, cust_Package_TO_SOT_SMD:SC-70, symbol PCM_Diode_AKL:BAV199W
- added R25, R26: 500k, Resistor_SMD:R_0603_1608Metric, symbol Device:R
- E1, E2: footprint (none) -> cust_Special_trace:Spark_Gap_1.65x1.1
- R5, R6: value 1.5Meg -> 1Meg
Connections:
- net GND: now also C10.2, C11.2, C12.2, C13.2, C14.2, C9.2, RV1.2
- net OUT+: now also D2.3 (C), R25.1; no longer R5.1
- net OUT-: now also D3.3 (C), R26.1; no longer R6.1
- net VCC: now also D2.2 (K), D3.2 (K)
- net VEE: now also D2.1 (A), D3.1 (A)
- new net: R25.2, R5.1
- new net: R26.2, R6.1
Other:
- note added: "C_parallel / C_series = R_series_1 / R_series_2 C_parallel = 5Meg / 102.0375k * 30p C_parallel = 147p"
- note added: "G_tot = [(R7+R8+R11)+RV1/2+(R1+R3+R5)] / [(R7+R8+R11)+RV1/2] G_tot = [102k+37.5+5Meg] / [102k+37.5] G_tot = 50.00159 G_tot =~ -34 dB"
- note removed: "G_tot = (R9+R10+R33+X1/2+R28+R27+R1) / (R9+R10+R33+X1/2) G_tot = (102k+37.5+5Meg) / (102k+37.5) G_tot = 50.00159 C_parallel / C_series = R_series / R_parallel C_parallel = 5Meg / 102.0375k * 30p C_parallel = 147p"
