File: DiffProbe.kicad_pcb (KiCad board)
At the start: 2 copper layers, 1 part

Commit message: Routed PCB
Parts:
- removed D1: BAV199DW, Package_TO_SOT_SMD:SOT-363_SC-70-6
- added C1: 12p, Capacitor_SMD:C_0603_1608Metric, F.Cu at (111.5, 63.2)
- added C10: 100p, Capacitor_SMD:C_0603_1608Metric, F.Cu at (126.0, 71.8)
- added C11: 30p, Capacitor_SMD:C_0603_1608Metric, F.Cu at (127.8, 64.0)
- added C12: 30p, Capacitor_SMD:C_0603_1608Metric, F.Cu at (127.8, 71.8)
- added C13: 17p (5-30p), Capacitor_SMD:C_Trimmer_Murata_TZB4-A, F.Cu at (132.6, 62.0)
- added C14: 17p (5-30p), Capacitor_SMD:C_Trimmer_Murata_TZB4-A, F.Cu at (132.6, 73.9)
- added C15: 1u, Capacitor_SMD:C_0603_1608Metric, F.Cu at (142.7, 69.3)
- added C17: 100p, Capacitor_SMD:C_0603_1608Metric, F.Cu at (145.8, 69.2)
- added C18: 100p, Capacitor_SMD:C_0603_1608Metric, F.Cu at (144.2, 69.2)
- added C19: 100p, Capacitor_SMD:C_0603_1608Metric, F.Cu at (143.5, 67.0)
- added C2: 12p, Capacitor_SMD:C_0603_1608Metric, F.Cu at (111.5, 72.6)
- added C20: 100p, Capacitor_SMD:C_0603_1608Metric, F.Cu at (143.5, 65.4)
- added C25: 0.1p, Capacitor_SMD:C_0603_1608Metric, F.Cu at (142.7, 61.5)
- added C26: 0.1p, Capacitor_SMD:C_0603_1608Metric, F.Cu at (142.5, 72.6)
- added C27: 1u, Capacitor_SMD:C_0603_1608Metric, F.Cu at (158.2, 74.2)
- added C28: 100p, Capacitor_SMD:C_0603_1608Metric, F.Cu at (155.2, 74.2)
- added C29: 100p, Capacitor_SMD:C_0603_1608Metric, F.Cu at (156.7, 74.2)
- added C3: 12p, Capacitor_SMD:C_0603_1608Metric, F.Cu at (114.8, 63.2)
- added C30: 100p, Capacitor_SMD:C_0603_1608Metric, F.Cu at (157.5, 76.5)
- added C31: 100p, Capacitor_SMD:C_0603_1608Metric, F.Cu at (157.5, 78.0)
- added C32: 0.1p, Capacitor_SMD:C_0603_1608Metric, F.Cu at (165.3, 74.7)
- added C33: 10u, Capacitor_SMD:C_0603_1608Metric, F.Cu at (164.0, 64.8)
- added C34: 10u, Capacitor_SMD:C_0603_1608Metric, F.Cu at (162.2, 64.8)
- added C35: 1u, Capacitor_SMD:C_0603_1608Metric, F.Cu at (160.4, 64.8)
- added C36: 100n, Capacitor_SMD:C_0603_1608Metric, F.Cu at (158.7, 64.8)
- added C37: C, Capacitor_SMD:C_0603_1608Metric, F.Cu at (152.7, 67.6)
- added C38: C, Capacitor_SMD:C_0603_1608Metric, F.Cu at (151.1, 63.1)
- added C39: C, Capacitor_SMD:C_0603_1608Metric, F.Cu at (151.1, 67.6)
- added C4: 12p, Capacitor_SMD:C_0603_1608Metric, F.Cu at (114.8, 72.6)
- added C40: C, Capacitor_SMD:C_0603_1608Metric, F.Cu at (152.7, 63.0)
- added C5: 12p, Capacitor_SMD:C_0603_1608Metric, F.Cu at (118.1, 63.2)
- added C6: 12p, Capacitor_SMD:C_0603_1608Metric, F.Cu at (118.1, 72.6)
- added C7: 12p, Capacitor_SMD:C_0603_1608Metric, F.Cu at (121.4, 63.2)
- added C8: 12p, Capacitor_SMD:C_0603_1608Metric, F.Cu at (121.4, 72.6)
- added C9: 100p, Capacitor_SMD:C_0603_1608Metric, F.Cu at (126.0, 64.0)
- added D2: BAV199W, cust_Package_TO_SOT_SMD:SC-70, F.Cu at (138.9, 60.2)
- added D3: BAV199W, cust_Package_TO_SOT_SMD:SC-70, F.Cu at (138.4, 75.9)
- added E1: SparkGap, cust_Special_trace:Spark_Gap_1.65x1.1, B.Cu at (110.9, 65.0)
- added E2: SparkGap, cust_Special_trace:Spark_Gap_1.65x1.1, B.Cu at (111.2, 70.9)
- added FB1: FerriteBead_Small, Inductor_SMD:L_0603_1608Metric, F.Cu at (163.2, 67.3)
- added FB2: FerriteBead_Small, Inductor_SMD:L_0603_1608Metric, F.Cu at (163.2, 62.3)
- added FB3: FerriteBead_Small, Inductor_SMD:L_0603_1608Metric, F.Cu at (151.9, 65.3)
- added J1: IN+, Connector_PinHeader_2.54mm:PinHeader_1x01_P2.54mm_Horizontal, F.Cu at (108.0, 65.0)
- added J2: IN-, Connector_PinHeader_2.54mm:PinHeader_1x01_P2.54mm_Horizontal, F.Cu at (108.0, 70.9)
- added J3: Conn_Coaxial, Connector_Coaxial:SMA_Samtec_SMA-J-P-X-ST-EM1_EdgeMount, F.Cu at (172.1, 75.5)
- added J4: USB_B_Micro, Connector_USB:USB_Micro-AB_Molex_47590-0001, F.Cu at (173.1, 64.8)
- added Q1: Q_PMOS_DGS, Package_TO_SOT_SMD:TSOT-23, F.Cu at (166.8, 64.8)
- added R1: 2Meg, Resistor_SMD:R_0603_1608Metric, F.Cu at (111.5, 65.0)
- added R10: 1k, Resistor_SMD:R_0603_1608Metric, F.Cu at (124.2, 71.8)
- added R11: 1k, Resistor_SMD:R_0603_1608Metric, F.Cu at (128.3, 66.5)
- added R12: 1k, Resistor_SMD:R_0603_1608Metric, F.Cu at (128.3, 69.1)
- added R13: 1k, Resistor_SMD:R_0603_1608Metric, F.Cu at (138.9, 63.8)
- added R14: 1k, Resistor_SMD:R_0603_1608Metric, F.Cu at (138.2, 71.9)
- added R15: 2k, Resistor_SMD:R_0603_1608Metric, F.Cu at (144.3, 61.5)
- added R16: 1k, Resistor_SMD:R_0603_1608Metric, F.Cu at (148.1, 71.9)
- added R17: 2k, Resistor_SMD:R_0603_1608Metric, F.Cu at (141.0, 72.6)
- added R18: 1k, Resistor_SMD:R_0603_1608Metric, F.Cu at (143.5, 63.8)
- added R19: 1k, Resistor_SMD:R_0603_1608Metric, F.Cu at (160.1, 71.9)
- added R2: 2Meg, Resistor_SMD:R_0603_1608Metric, F.Cu at (111.5, 70.9)
- added R20: 1k, Resistor_SMD:R_0603_1608Metric, F.Cu at (145.8, 64.5)
- added R21: 1k, Resistor_SMD:R_0603_1608Metric, F.Cu at (163.8, 74.7)
- added R22: 50, Resistor_SMD:R_0603_1608Metric, F.Cu at (167.8, 75.5)
- added R23: R, Resistor_SMD:R_0603_1608Metric, F.Cu at (158.7, 68.2)
- added R24: R, Resistor_SMD:R_0603_1608Metric, F.Cu at (158.7, 61.4)
- added R25: 500k, Resistor_SMD:R_0603_1608Metric, F.Cu at (121.4, 65.0)
- added R26: 500k, Resistor_SMD:R_0603_1608Metric, F.Cu at (121.4, 70.9)
- added R3: 1.5Meg, Resistor_SMD:R_0603_1608Metric, F.Cu at (114.8, 65.0)
- added R4: 1.5Meg, Resistor_SMD:R_0603_1608Metric, F.Cu at (114.8, 70.9)
- added R5: 1Meg, Resistor_SMD:R_0603_1608Metric, F.Cu at (118.1, 65.0)
- added R6: 1Meg, Resistor_SMD:R_0603_1608Metric, F.Cu at (118.1, 70.9)
- added R7: 1k, Resistor_SMD:R_0603_1608Metric, F.Cu at (124.2, 64.0)
- added R8: 100k, Resistor_SMD:R_0603_1608Metric, F.Cu at (125.0, 66.5)
- added R9: 100k, Resistor_SMD:R_0603_1608Metric, F.Cu at (125.0, 69.1)
- added RV1: 75R, Potentiometer_SMD:Potentiometer_Bourns_3214W_Vertical, F.Cu at (132.5, 67.8)
- added U1: LTC6269 A, Package_SO:MSOP-8-1EP_3x3mm_P0.65mm_EP1.68x1.88mm, F.Cu at (140.2, 67.8)
- added U3: LTC6268IS6, Package_TO_SOT_SMD:TSOT-23-6, F.Cu at (161.0, 75.0)
- added U4: any (e.g. LM7301), Package_SO:MSOP-8_3x3mm_P0.65mm, F.Cu at (155.9, 64.9)
Routing:
- net VEE: track 0.00 -> 78.5 mm, vias 0 -> 2
- net VCC: track 0.00 -> 61.1 mm, vias 0 -> 4
- net GND: track 0.00 -> 56.8 mm, vias 0 -> 24
- net Net-(U3-+): track 0.00 -> 32.5 mm, vias 0 -> 2
- net Net-(C26-Pad1): track 0.00 -> 20.3 mm
- net Net-(U1A--): track 0.00 -> 20.3 mm
- net Net-(U4B-+): track 0.00 -> 19.1 mm, vias 0 -> 2
- net /Atternuator/OUT-: track 0.00 -> 14.6 mm
- net /Atternuator/OUT+: track 0.00 -> 14.5 mm
- net Net-(U1B--): track 0.00 -> 12.0 mm
- net /Gain stage/OUT: track 0.00 -> 8.13 mm
- net /Atternuator/IN-: track 0.00 -> 7.99 mm
- net /Atternuator/IN+: track 0.00 -> 6.98 mm
- net Net-(C25-Pad1): track 0.00 -> 6.17 mm
- net Net-(U3--): track 0.00 -> 6.10 mm
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- added copper zone on F.Cu, net /Atternuator/OUT+
- added copper zone on F.Cu, net /Atternuator/OUT-
- added copper zone on B.Cu, net GND
- added copper zone on F.Cu, net GND
- added copper zone on F.Cu, net Net-(J4-GND)
- added copper zone on F.Cu, net Net-(Q1-S)
- added copper zone on F.Cu, net Net-(U4B--)
- added copper zone on F.Cu, net VCC
- added copper zone on F.Cu, net VEE
Other:
- board outline added: 68.1 x 22.9 mm
- board text added: "IN+"
- board text added: "IN-"
