File: DiffProbe.kicad_sch (KiCad schematic)
At the start: 4 parts, among them J1 IN+, J2 IN-, J3 Conn_Coaxial

Commit message: Routed PCB
Parts:
- J1, J2: footprint Connector_PinHeader_1.00mm:PinHeader_1x01_P1.00mm_Horizontal -> Connector_PinHeader_2.54mm:PinHeader_1x01_P2.54mm_Horizontal; symbol Connector:Conn_01x01_Male -> Connector:Conn_01x01_Pin
Other:
- note added: "Differential gain: 1/10 Input impedance: 5Meg // 3pF Common-mode range: 70Vac Differential range: +-25V @ 70Vac common-mode Bandwidth ~ 100 MHz"
