File: Power.kicad_sch (KiCad schematic)
At the start: 16 parts, among them J4 USB_B_Micro, Q1 Q_PMOS_DGS, U4 any (e.g. LM7301)

Commit message: Routed PCB
Parts:
- added unit 3 of U4
- added unit 1 of U4
- U4: footprint Package_SO:SOIC-8-1EP_3.9x4.9mm_P1.27mm_EP2.29x3mm -> Package_SO:MSOP-8_3x3mm_P0.65mm; symbol pspice:OPAMP -> Amplifier_Operational:TL072
Connections:
- net VCC: now also U4.8 (V+); no longer U4.4 (V+)
- net VEE: now also U4.4 (V-); no longer U4.5 (V-)
- net at R23.2, R24.1: now also U4.5 (+); no longer U4.1 (+)
- new net: FB3.1, U4.6 (-), U4.7
- no-connect marks 3 -> 6
Other:
- note added: "Split rail supply +5 > +-2.5V"
- moved on the sheet: FB3
